Commit message: #2; create localbot packages based on softbot

File: localbot_description/urdf/VLP-16.urdf.xacro (robot description, xacro)
@@ -11,6 +11,5 @@
       <inertial>
 <!--        <mass value="0.83"/>-->
-<!--        <mass value="0.083"/>-->
-        <mass value="0.0"/>
+        <mass value="0.083"/>
         <origin xyz="0 0 0.03585"/>
         <inertia ixx="${(0.83 * (3.0*0.0516*0.0516 + 0.0717*0.0717)) / 12.0}" ixy="0" ixz="0"
@@ -59,5 +58,5 @@
         <sensor type="gpu_ray" name="${name}-VLP16">
           <pose>0 0 0 0 0 0</pose>
-          <visualize>true</visualize>
+          <visualize>false</visualize>
           <update_rate>${hz}</update_rate>
           <ray>

File: localbot_description/urdf/astra.urdf.xacro (robot description, xacro)
@@ -29,6 +29,5 @@
       <inertial>
 <!--        <mass value="0.564" />-->
-<!--        <mass value="0.00564" />-->
-          <mass value="0.0" />
+        <mass value="0.00564" />
         <origin xyz="0 0 0" />
         <inertia ixx="0.003881243" ixy="0.0" ixz="0.0"

File: localbot_description/urdf/localbot.gazebo.macro.xacro (robot description, xacro)
@@ -1,16 +1,18 @@
 <?xml version="1.0"?>
-<robot name="localbot" xmlns:xacro="http://ros.org/wiki/xacro">
-  <xacro:include filename="$(find localbot_description)/urdf/ros_diff_drive.gazebo.xacro"/>
-  <!--<xacro:include filename="$(find localbot_description)/urdf/ros_control.gazebo.xacro"/>-->
-  <xacro:arg name="laser_visual"  default="false"/>
-  <xacro:arg name="camera_visual" default="false"/>
-  <xacro:arg name="imu_visual"    default="false"/>
+<robot name="gazebo_macro" xmlns:xacro="http://ros.org/wiki/xacro">
+<xacro:macro name="gazebo_macro" params="color laser_visual camera_visual imu_visual">
+<!--  <xacro:arg name="laser_visual"  default="false"/>-->
+<!--  <xacro:arg name="camera_visual" default="false"/>-->
+<!--  <xacro:arg name="imu_visual"    default="false"/>-->
   <gazebo reference="base_link">
+<!--    <material>Gazebo/DarkGrey</material>-->
     <material>Gazebo/${color}</material>
-        <sensor name="base_link" type="contact">
+  </gazebo>
+  <gazebo reference="base_link">
+    <sensor name="base_link" type="contact">
       <update_rate>1000.0</update_rate>
       <always_on>true</always_on>
       <contact>
-        <collision>base_footprint_fixed_joint_lump__base_link_collision</collision>
+        <collision>base_footprint_fixed_joint_lump__base_link_collision_collision</collision>
       </contact>
       <plugin name="base_link_contact_sensor_plugin" filename="libgazebo_ros_bumper.so">
@@ -28,4 +30,5 @@
     <maxVel>0.1</maxVel>
     <fdir1>1 0 0</fdir1>
+    <!--    Gazebo properties are global: https://answers.ros.org/question/216975/loading-variables-with-xacroinclude/ -->
     <material>Gazebo/${color}</material>
   </gazebo>
@@ -36,7 +39,8 @@
     <kd>10.0</kd>
     <minDepth>0.001</minDepth>
-    <maxVel>0.1</maxVel>
+    <maxVel>0.01</maxVel>
     <fdir1>1 0 0</fdir1>
-   <material>Gazebo/${color}</material>
+    <!--    Gazebo properties are global: https://answers.ros.org/question/216975/loading-variables-with-xacroinclude/ -->
+    <material>Gazebo/${color}</material>
   </gazebo>
   <gazebo reference="caster_back_right_link">
@@ -61,10 +65,10 @@
     <sensor type="imu" name="imu">
       <always_on>true</always_on>
-      <visualize>$(arg imu_visual)</visualize>
+      <visualize>${imu_visual}</visualize>
     </sensor>
     <material>Gazebo/Grey</material>
   </gazebo>
   <!--Using gazebo or ROS native controller for differential drives.-->
-  <!-- <xacro:include filename="$(find localbot_description)/urdf/ros_diff_drive.gazebo.xacro"/> -->
+  <xacro:include filename="$(find localbot_description)/urdf/ros_diff_drive.gazebo.xacro"/>
   <gazebo>
     <plugin name="imu_plugin" filename="libgazebo_ros_imu.so">
@@ -95,3 +99,37 @@
     </plugin>
   </gazebo>
+  <gazebo reference="base_scan">
+    <material>Gazebo/FlatBlack</material>
+    <sensor type="ray" name="lds_lfcd_sensor">
+      <pose>0 0 0 0 0 0</pose>
+      <visualize>${laser_visual}</visualize>
+<!--      <visualize>true</visualize>-->
+      <update_rate>5</update_rate>
+      <ray>
+        <scan>
+          <horizontal>
+            <samples>360</samples>
+            <resolution>1</resolution>
+            <min_angle>0.0</min_angle>
+            <max_angle>6.28319</max_angle>
+          </horizontal>
+        </scan>
+        <range>
+          <min>0.120</min>
+          <max>3.5</max>
+          <resolution>0.015</resolution>
+        </range>
+        <noise>
+          <type>gaussian</type>
+          <mean>0.0</mean>
+          <stddev>0.01</stddev>
+        </noise>
+      </ray>
+      <plugin name="gazebo_ros_lds_lfcd_controller" filename="libgazebo_ros_laser.so">
+        <topicName>scan</topicName>
+        <frameName>base_scan</frameName>
+      </plugin>
+    </sensor>
+  </gazebo>
+</xacro:macro>
 </robot>

File: localbot_description/urdf/localbot.urdf.xacro (robot description, xacro)
@@ -1,5 +1,12 @@
 <?xml version="1.0" ?>
 <robot name="localbot" xmlns:xacro="http://ros.org/wiki/xacro">
-  <xacro:include filename="$(find localbot_description)/urdf/common_properties.xacro"/>
+  <!--  Xacro description of turtlebot robot waffle pi used to play team hunt.-->
+  <!--  Miguel Riem Oliveira-->
+  <!--  PARI, November 2020-->
+  <!--Args are local, properties are global, so we copy the values of the arguments to the properties-->
+  <xacro:arg name="name" default="localbot" />
+  <xacro:arg name="color" default="Orange" /> <!-- e.g. Red, Orange. Must exist in Gazebo/Colors and be defined in properties.xacro.-->
+  <!--Properties are global so they can be viewed from inside the included xacros-->
+  <!--  args are used with $(arg arg_name), properties are used as ${property_name}-->
   <xacro:property name="name" value="$(arg name)"/>
   <xacro:property name="color" value="$(arg color)"/>
@@ -8,6 +15,7 @@
   <xacro:include filename="$(find localbot_description)/urdf/VLP-16.urdf.xacro"/>
   <xacro:include filename="$(find localbot_description)/urdf/astra.urdf.xacro" />
-  <xacro:include filename="$(find velodyne_description)/urdf/VLP-16.urdf.xacro"/>
   <xacro:include filename="$(find localbot_description)/urdf/localbot.gazebo.macro.xacro"/>
+  <xacro:gazebo_macro color="$(arg color)" laser_visual="false" camera_visual="false" imu_visual="true"/>
+  <!-- Links and joints-->
   <link name="base_footprint"/>
   <joint name="base_joint" type="fixed">
@@ -22,10 +30,11 @@
         <mesh filename="package://turtlebot3_description/meshes/bases/waffle_pi_base.stl" scale="0.001 0.001 0.001"/>
       </geometry>
-      <material name="Grey"/>
-    </visual>
-    <collision>
-      <origin xyz="-0.064 0 0.047" rpy="0 0 0.5"/>
-      <geometry>
-        <box size="0.266 0.266 0.094"/>
+      <material name="light_black"/>
+    </visual>
+    <collision name="base_link_collision">
+      <origin xyz="-0.064 0 0.047" rpy="0 0 0"/>
+      <geometry>
+        <!--        <box size="0.266 0.266 0.094"/>-->
+        <box size="0.3 0.3 0.094"/>
       </geometry>
     </collision>
@@ -50,5 +59,5 @@
         <mesh filename="package://turtlebot3_description/meshes/wheels/left_tire.stl" scale="0.001 0.001 0.001"/>
       </geometry>
-      <material name="Grey"/>
+      <material name="black"/>
     </visual>
     <collision>
@@ -64,5 +73,5 @@
                iyy="1.1192413e-05" iyz="-1.4400107e-11"
                izz="2.0712558e-05" />
-      </inertial>
+    </inertial>
   </link>
   <joint name="wheel_right_joint" type="continuous">
@@ -78,6 +87,5 @@
         <mesh filename="package://turtlebot3_description/meshes/wheels/right_tire.stl" scale="0.001 0.001 0.001"/>
       </geometry>
-<!--      <material name="Grey"/>-->
-      <material name="Grey"/>
+      <material name="black"/>
     </visual>
     <collision>
@@ -93,5 +101,5 @@
                iyy="1.1192413e-05" iyz="-1.4400107e-11"
                izz="2.0712558e-05" />
-      </inertial>
+    </inertial>
   </link>
   <joint name="caster_back_right_joint" type="fixed">
@@ -141,17 +149,106 @@
   </joint>
   <link name="imu_link"/>
-  </robot>
-  <!-- <link name="camera_support_link">
-  </link>
-  <joint name="platform_support_camera_link" type="fixed">
-    <origin xyz="0.02 0 1.5" rpy="0.01 -0.35 0.2"/>
-    <parent link="base_link"/>
-    <child link="camera_support_link"/>
-  </joint>
-  <xacro:sensor_astra prefix="camera" parent="camera_support_link">
+  <link name="platform_support_leg1_link">
+    <visual>
+      <origin xyz="0 0 -0.1" rpy="0 0 0"/>
+      <geometry>
+        <cylinder length="0.2" radius="0.004"/>
+      </geometry>
+      <material name="grey"/>
+    </visual>
+  </link>
+  <joint name="base_link_to_platform_support_leg1_link" type="fixed">
+    <parent link="base_link"/>
+    <child link="platform_support_leg1_link"/>
+    <origin xyz="-0.114 0.05 0.222" rpy="0 0 0"/>
+  </joint>
+  <link name="platform_support_leg2_link">
+    <visual>
+      <origin xyz="0 0 -0.1" rpy="0 0 0"/>
+      <geometry>
+        <cylinder length="0.2" radius="0.004"/>
+      </geometry>
+      <material name="grey"/>
+    </visual>
+  </link>
+  <joint name="base_link_to_platform_support_leg2_link" type="fixed">
+    <parent link="base_link"/>
+    <child link="platform_support_leg2_link"/>
+    <origin xyz="-0.114 -0.05 0.222" rpy="0 0 0"/>
+  </joint>
+  <link name="platform_support_leg3_link">
+    <visual>
+      <origin xyz="0 0 -0.1" rpy="0 0 0"/>
+      <geometry>
+        <cylinder length="0.2" radius="0.004"/>
+      </geometry>
+      <material name="grey"/>
+    </visual>
+  </link>
+  <joint name="base_link_to_platform_support_leg3_link" type="fixed">
+    <parent link="base_link"/>
+    <child link="platform_support_leg3_link"/>
+    <origin xyz="-0.014 0.05 0.222" rpy="0 0 0"/>
+  </joint>
+  <link name="platform_support_leg4_link">
+    <visual>
+      <origin xyz="0 0 -0.1" rpy="0 0 0"/>
+      <geometry>
+        <cylinder length="0.2" radius="0.004"/>
+      </geometry>
+      <material name="grey"/>
+    </visual>
+  </link>
+  <joint name="base_link_to_platform_support_leg4_link" type="fixed">
+    <parent link="base_link"/>
+    <child link="platform_support_leg4_link"/>
+    <origin xyz="-0.014 -0.05 0.222" rpy="0 0 0"/>
+  </joint>
+  <link name="lidar3d_plate_link">
+    <visual>
+      <origin xyz="0 0 0" rpy="0 0 0"/>
+      <geometry>
+        <box size="0.14 0.14 0.005"/>
+      </geometry>
+      <material name="grey"/>
+    </visual>
+  </link>
+  <joint name="platform_support_leg1_link_to_lidar3d_plate_link" type="fixed">
+    <parent link="platform_support_leg1_link"/>
+    <child link="lidar3d_plate_link"/>
+    <origin xyz="0.05 -0.05 0" rpy="0 0 0"/>
+  </joint>
+  <xacro:VLP-16 name="lidar3d" parent="lidar3d_plate_link" topic="/lidar3d/points">
+    <origin xyz="0 0 0" rpy="0 0 0" />
+  </xacro:VLP-16>
+  <link name="front_left_camera_support_link">
+  </link>
+  <joint name="platform_support_leg3_link_to_front_left_camera_support_link" type="fixed">
+    <origin xyz="0.02 0 -0.09" rpy="0.01 -0.35 0.2"/>
+    <parent link="platform_support_leg3_link"/>
+    <child link="front_left_camera_support_link"/>
+  </joint>
+  <xacro:sensor_astra prefix="front_left_camera" parent="front_left_camera_support_link">
     <origin xyz="0.02 0.07 0.015" rpy="0 0.0 0" />
   </xacro:sensor_astra>
-    3d lidar
-  <xacro:VLP-16 name="lidar3d" parent="base_link" topic="/lidar3d/points">
-        <origin xyz="0 0 0.7" rpy="0 0 0" />
-  </xacro:VLP-16> -->
+  <link name="front_right_camera_support_link">
+  </link>
+  <joint name="platform_support_leg4_link_to_front_right_camera_support_link" type="fixed">
+    <origin xyz="0.02 0 -0.05" rpy="0.01 -0.35 -0.22"/>
+    <parent link="platform_support_leg4_link"/>
+    <child link="front_right_camera_support_link"/>
+  </joint>
+  <xacro:sensor_astra prefix="front_right_camera" parent="front_right_camera_support_link">
+    <origin xyz="0.02 0.07 0.015" rpy="0 0.0 0" />
+  </xacro:sensor_astra>
+  <link name="back_camera_support_link">
+  </link>
+  <joint name="platform_support_leg1_link_to_back_camera_support_link" type="fixed">
+    <origin xyz="-0.02 -0.05 -0.10" rpy="0.01 -0.35 3.14"/>
+    <parent link="platform_support_leg1_link"/>
+    <child link="back_camera_support_link"/>
+  </joint>
+  <xacro:sensor_astra prefix="back_camera" parent="back_camera_support_link">
+    <origin xyz="0.02 0.07 0.015" rpy="0 0.0 0" />
+  </xacro:sensor_astra>
+</robot>
