Commit message: #4; update localbot to contain only one RGBD camera

File: localbot_description/urdf/localbot.gazebo.macro.xacro (robot description, xacro)
@@ -5,14 +5,15 @@
 <!--  <xacro:arg name="camera_visual" default="false"/>-->
 <!--  <xacro:arg name="imu_visual"    default="false"/>-->
-  <gazebo reference="base_link">
+  <gazebo reference="camera_support_kink">
 <!--    <material>Gazebo/DarkGrey</material>-->
     <material>Gazebo/${color}</material>
   </gazebo>
-  <gazebo reference="base_link">
-    <sensor name="base_link" type="contact">
+  <gazebo reference="camera_support_link">
+  <gravity>0</gravity>
+    <sensor name="camera_support_link" type="contact">
       <update_rate>1000.0</update_rate>
       <always_on>true</always_on>
       <contact>
-        <collision>base_footprint_fixed_joint_lump__base_link_collision_collision</collision>
+        <collision>camera_support_link_contact</collision>
       </contact>
       <plugin name="base_link_contact_sensor_plugin" filename="libgazebo_ros_bumper.so">
@@ -22,114 +23,4 @@
     </sensor>
   </gazebo>
-  <gazebo reference="wheel_left_link">
-    <mu1>0.1</mu1>
-    <mu2>0.1</mu2>
-    <kp>500000.0</kp>
-    <kd>10.0</kd>
-    <minDepth>0.001</minDepth>
-    <maxVel>0.1</maxVel>
-    <fdir1>1 0 0</fdir1>
-    <!--    Gazebo properties are global: https://answers.ros.org/question/216975/loading-variables-with-xacroinclude/ -->
-    <material>Gazebo/${color}</material>
-  </gazebo>
-  <gazebo reference="wheel_right_link">
-    <mu1>0.1</mu1>
-    <mu2>0.1</mu2>
-    <kp>500000.0</kp>
-    <kd>10.0</kd>
-    <minDepth>0.001</minDepth>
-    <maxVel>0.01</maxVel>
-    <fdir1>1 0 0</fdir1>
-    <!--    Gazebo properties are global: https://answers.ros.org/question/216975/loading-variables-with-xacroinclude/ -->
-    <material>Gazebo/${color}</material>
-  </gazebo>
-  <gazebo reference="caster_back_right_link">
-    <mu1>0.1</mu1>
-    <mu2>0.1</mu2>
-    <kp>1000000.0</kp>
-    <kd>100.0</kd>
-    <minDepth>0.001</minDepth>
-    <maxVel>1.0</maxVel>
-    <material>Gazebo/FlatBlack</material>
-  </gazebo>
-  <gazebo reference="caster_back_left_link">
-    <mu1>0.1</mu1>
-    <mu2>0.1</mu2>
-    <kp>1000000.0</kp>
-    <kd>100.0</kd>
-    <minDepth>0.001</minDepth>
-    <maxVel>1.0</maxVel>
-    <material>Gazebo/FlatBlack</material>
-  </gazebo>
-  <gazebo reference="imu_link">
-    <sensor type="imu" name="imu">
-      <always_on>true</always_on>
-      <visualize>${imu_visual}</visualize>
-    </sensor>
-    <material>Gazebo/Grey</material>
-  </gazebo>
-  <!--Using gazebo or ROS native controller for differential drives.-->
-  <xacro:include filename="$(find localbot_description)/urdf/ros_diff_drive.gazebo.xacro"/>
-  <gazebo>
-    <plugin name="imu_plugin" filename="libgazebo_ros_imu.so">
-      <alwaysOn>true</alwaysOn>
-      <bodyName>imu_link</bodyName>
-      <frameName>imu_link</frameName>
-      <topicName>imu</topicName>
-      <serviceName>imu_service</serviceName>
-      <gaussianNoise>0.0</gaussianNoise>
-      <updateRate>200</updateRate>
-      <imu>
-        <noise>
-          <type>gaussian</type>
-          <rate>
-            <mean>0.0</mean>
-            <stddev>2e-4</stddev>
-            <bias_mean>0.0000075</bias_mean>
-            <bias_stddev>0.0000008</bias_stddev>
-          </rate>
-          <accel>
-            <mean>0.0</mean>
-            <stddev>1.7e-2</stddev>
-            <bias_mean>0.1</bias_mean>
-            <bias_stddev>0.001</bias_stddev>
-          </accel>
-        </noise>
-      </imu>
-    </plugin>
-  </gazebo>
-  <gazebo reference="base_scan">
-    <material>Gazebo/FlatBlack</material>
-    <sensor type="ray" name="lds_lfcd_sensor">
-      <pose>0 0 0 0 0 0</pose>
-      <visualize>${laser_visual}</visualize>
-<!--      <visualize>true</visualize>-->
-      <update_rate>5</update_rate>
-      <ray>
-        <scan>
-          <horizontal>
-            <samples>360</samples>
-            <resolution>1</resolution>
-            <min_angle>0.0</min_angle>
-            <max_angle>6.28319</max_angle>
-          </horizontal>
-        </scan>
-        <range>
-          <min>0.120</min>
-          <max>3.5</max>
-          <resolution>0.015</resolution>
-        </range>
-        <noise>
-          <type>gaussian</type>
-          <mean>0.0</mean>
-          <stddev>0.01</stddev>
-        </noise>
-      </ray>
-      <plugin name="gazebo_ros_lds_lfcd_controller" filename="libgazebo_ros_laser.so">
-        <topicName>scan</topicName>
-        <frameName>base_scan</frameName>
-      </plugin>
-    </sensor>
-  </gazebo>
 </xacro:macro>
 </robot>

File: localbot_description/urdf/localbot.urdf.xacro (robot description, xacro)
@@ -17,238 +17,8 @@
   <xacro:include filename="$(find localbot_description)/urdf/localbot.gazebo.macro.xacro"/>
   <xacro:gazebo_macro color="$(arg color)" laser_visual="false" camera_visual="false" imu_visual="true"/>
-  <!-- Links and joints-->
-  <link name="base_footprint"/>
-  <joint name="base_joint" type="fixed">
-    <parent link="base_footprint"/>
-    <child link="base_link" />
-    <origin xyz="0 0 0.010" rpy="0 0 0"/>
-  </joint>
-  <link name="base_link">
-    <visual>
-      <origin xyz="-0.064 0 0.0" rpy="0 0 0"/>
-      <geometry>
-        <mesh filename="package://turtlebot3_description/meshes/bases/waffle_pi_base.stl" scale="0.001 0.001 0.001"/>
-      </geometry>
-      <material name="light_black"/>
-    </visual>
-    <collision name="base_link_collision">
-      <origin xyz="-0.064 0 0.047" rpy="0 0 0"/>
-      <geometry>
-        <!--        <box size="0.266 0.266 0.094"/>-->
-        <box size="0.3 0.3 0.094"/>
-      </geometry>
-    </collision>
-    <inertial>
-      <origin xyz="0 0 0" rpy="0 0 0"/>
-      <mass value="1.3729096e+00"/>
-      <inertia ixx="8.7002718e-03" ixy="-4.7576583e-05" ixz="1.1160499e-04"
-               iyy="8.6195418e-03" iyz="-3.5422299e-06"
-               izz="1.4612727e-02" />
-    </inertial>
+  <link name="camera_support_link">
   </link>
-  <joint name="wheel_left_joint" type="continuous">
-    <parent link="base_link"/>
-    <child link="wheel_left_link"/>
-    <origin xyz="0.0 0.144 0.023" rpy="-1.57 0 0"/>
-    <axis xyz="0 0 1"/>
-  </joint>
-  <link name="wheel_left_link">
-    <visual>
-      <origin xyz="0 0 0" rpy="1.57 0 0"/>
-      <geometry>
-        <mesh filename="package://turtlebot3_description/meshes/wheels/left_tire.stl" scale="0.001 0.001 0.001"/>
-      </geometry>
-      <material name="black"/>
-    </visual>
-    <collision>
-      <origin xyz="0 0 0" rpy="0 0 0"/>
-      <geometry>
-        <cylinder length="0.018" radius="0.033"/>
-      </geometry>
-    </collision>
-    <inertial>
-      <origin xyz="0 0 0" />
-      <mass value="2.8498940e-02" />
-      <inertia ixx="1.1175580e-05" ixy="-4.2369783e-11" ixz="-5.9381719e-09"
-               iyy="1.1192413e-05" iyz="-1.4400107e-11"
-               izz="2.0712558e-05" />
-    </inertial>
-  </link>
-  <joint name="wheel_right_joint" type="continuous">
-    <parent link="base_link"/>
-    <child link="wheel_right_link"/>
-    <origin xyz="0.0 -0.144 0.023" rpy="-1.57 0 0"/>
-    <axis xyz="0 0 1"/>
-  </joint>
-  <link name="wheel_right_link">
-    <visual>
-      <origin xyz="0 0 0" rpy="1.57 0 0"/>
-      <geometry>
-        <mesh filename="package://turtlebot3_description/meshes/wheels/right_tire.stl" scale="0.001 0.001 0.001"/>
-      </geometry>
-      <material name="black"/>
-    </visual>
-    <collision>
-      <origin xyz="0 0 0" rpy="0 0 0"/>
-      <geometry>
-        <cylinder length="0.018" radius="0.033"/>
-      </geometry>
-    </collision>
-    <inertial>
-      <origin xyz="0 0 0" />
-      <mass value="2.8498940e-02" />
-      <inertia ixx="1.1175580e-05" ixy="-4.2369783e-11" ixz="-5.9381719e-09"
-               iyy="1.1192413e-05" iyz="-1.4400107e-11"
-               izz="2.0712558e-05" />
-    </inertial>
-  </link>
-  <joint name="caster_back_right_joint" type="fixed">
-    <parent link="base_link"/>
-    <child link="caster_back_right_link"/>
-    <origin xyz="-0.177 -0.064 -0.004" rpy="-1.57 0 0"/>
-  </joint>
-  <link name="caster_back_right_link">
-    <collision>
-      <origin xyz="0 0.001 0" rpy="0 0 0"/>
-      <geometry>
-        <box size="0.030 0.009 0.020"/>
-      </geometry>
-    </collision>
-    <inertial>
-      <origin xyz="0 0 0" />
-      <mass value="0.005" />
-      <inertia ixx="0.001" ixy="0.0" ixz="0.0"
-               iyy="0.001" iyz="0.0"
-               izz="0.001" />
-    </inertial>
-  </link>
-  <joint name="caster_back_left_joint" type="fixed">
-    <parent link="base_link"/>
-    <child link="caster_back_left_link"/>
-    <origin xyz="-0.177 0.064 -0.004" rpy="-1.57 0 0"/>
-  </joint>
-  <link name="caster_back_left_link">
-    <collision>
-      <origin xyz="0 0.001 0" rpy="0 0 0"/>
-      <geometry>
-        <box size="0.030 0.009 0.020"/>
-      </geometry>
-    </collision>
-    <inertial>
-      <origin xyz="0 0 0" />
-      <mass value="0.005" />
-      <inertia ixx="0.001" ixy="0.0" ixz="0.0"
-               iyy="0.001" iyz="0.0"
-               izz="0.001" />
-    </inertial>
-  </link>
-  <joint name="imu_joint" type="fixed">
-    <parent link="base_link"/>
-    <child link="imu_link"/>
-    <origin xyz="0.0 0 0.068" rpy="0 0 0"/>
-  </joint>
-  <link name="imu_link"/>
-  <link name="platform_support_leg1_link">
-    <visual>
-      <origin xyz="0 0 -0.1" rpy="0 0 0"/>
-      <geometry>
-        <cylinder length="0.2" radius="0.004"/>
-      </geometry>
-      <material name="grey"/>
-    </visual>
-  </link>
-  <joint name="base_link_to_platform_support_leg1_link" type="fixed">
-    <parent link="base_link"/>
-    <child link="platform_support_leg1_link"/>
-    <origin xyz="-0.114 0.05 0.222" rpy="0 0 0"/>
-  </joint>
-  <link name="platform_support_leg2_link">
-    <visual>
-      <origin xyz="0 0 -0.1" rpy="0 0 0"/>
-      <geometry>
-        <cylinder length="0.2" radius="0.004"/>
-      </geometry>
-      <material name="grey"/>
-    </visual>
-  </link>
-  <joint name="base_link_to_platform_support_leg2_link" type="fixed">
-    <parent link="base_link"/>
-    <child link="platform_support_leg2_link"/>
-    <origin xyz="-0.114 -0.05 0.222" rpy="0 0 0"/>
-  </joint>
-  <link name="platform_support_leg3_link">
-    <visual>
-      <origin xyz="0 0 -0.1" rpy="0 0 0"/>
-      <geometry>
-        <cylinder length="0.2" radius="0.004"/>
-      </geometry>
-      <material name="grey"/>
-    </visual>
-  </link>
-  <joint name="base_link_to_platform_support_leg3_link" type="fixed">
-    <parent link="base_link"/>
-    <child link="platform_support_leg3_link"/>
-    <origin xyz="-0.014 0.05 0.222" rpy="0 0 0"/>
-  </joint>
-  <link name="platform_support_leg4_link">
-    <visual>
-      <origin xyz="0 0 -0.1" rpy="0 0 0"/>
-      <geometry>
-        <cylinder length="0.2" radius="0.004"/>
-      </geometry>
-      <material name="grey"/>
-    </visual>
-  </link>
-  <joint name="base_link_to_platform_support_leg4_link" type="fixed">
-    <parent link="base_link"/>
-    <child link="platform_support_leg4_link"/>
-    <origin xyz="-0.014 -0.05 0.222" rpy="0 0 0"/>
-  </joint>
-  <link name="lidar3d_plate_link">
-    <visual>
-      <origin xyz="0 0 0" rpy="0 0 0"/>
-      <geometry>
-        <box size="0.14 0.14 0.005"/>
-      </geometry>
-      <material name="grey"/>
-    </visual>
-  </link>
-  <joint name="platform_support_leg1_link_to_lidar3d_plate_link" type="fixed">
-    <parent link="platform_support_leg1_link"/>
-    <child link="lidar3d_plate_link"/>
-    <origin xyz="0.05 -0.05 0" rpy="0 0 0"/>
-  </joint>
-  <xacro:VLP-16 name="lidar3d" parent="lidar3d_plate_link" topic="/lidar3d/points">
-    <origin xyz="0 0 0" rpy="0 0 0" />
-  </xacro:VLP-16>
-  <link name="front_left_camera_support_link">
-  </link>
-  <joint name="platform_support_leg3_link_to_front_left_camera_support_link" type="fixed">
-    <origin xyz="0.02 0 -0.09" rpy="0.01 -0.35 0.2"/>
-    <parent link="platform_support_leg3_link"/>
-    <child link="front_left_camera_support_link"/>
-  </joint>
-  <xacro:sensor_astra prefix="front_left_camera" parent="front_left_camera_support_link">
-    <origin xyz="0.02 0.07 0.015" rpy="0 0.0 0" />
-  </xacro:sensor_astra>
-  <link name="front_right_camera_support_link">
-  </link>
-  <joint name="platform_support_leg4_link_to_front_right_camera_support_link" type="fixed">
-    <origin xyz="0.02 0 -0.05" rpy="0.01 -0.35 -0.22"/>
-    <parent link="platform_support_leg4_link"/>
-    <child link="front_right_camera_support_link"/>
-  </joint>
-  <xacro:sensor_astra prefix="front_right_camera" parent="front_right_camera_support_link">
-    <origin xyz="0.02 0.07 0.015" rpy="0 0.0 0" />
-  </xacro:sensor_astra>
-  <link name="back_camera_support_link">
-  </link>
-  <joint name="platform_support_leg1_link_to_back_camera_support_link" type="fixed">
-    <origin xyz="-0.02 -0.05 -0.10" rpy="0.01 -0.35 3.14"/>
-    <parent link="platform_support_leg1_link"/>
-    <child link="back_camera_support_link"/>
-  </joint>
-  <xacro:sensor_astra prefix="back_camera" parent="back_camera_support_link">
-    <origin xyz="0.02 0.07 0.015" rpy="0 0.0 0" />
+  <xacro:sensor_astra prefix="camera" parent="camera_support_link">
+    <origin xyz="0.00 0.00 1.00" rpy="0 0.0 0" />
   </xacro:sensor_astra>
 </robot>

Commit message: update rviz config file and add base_footprint link

File: localbot_description/urdf/localbot.gazebo.macro.xacro (robot description, xacro)
@@ -5,15 +5,15 @@
 <!--  <xacro:arg name="camera_visual" default="false"/>-->
 <!--  <xacro:arg name="imu_visual"    default="false"/>-->
-  <gazebo reference="camera_support_kink">
+  <gazebo reference="base_footprint">
 <!--    <material>Gazebo/DarkGrey</material>-->
     <material>Gazebo/${color}</material>
   </gazebo>
-  <gazebo reference="camera_support_link">
+  <gazebo reference="base_link">
   <gravity>0</gravity>
-    <sensor name="camera_support_link" type="contact">
+    <sensor name="base_link" type="contact">
       <update_rate>1000.0</update_rate>
       <always_on>true</always_on>
       <contact>
-        <collision>camera_support_link_contact</collision>
+        <collision>base_footprint_fixed_joint_lump__base_link_collision_collision</collision>
       </contact>
       <plugin name="base_link_contact_sensor_plugin" filename="libgazebo_ros_bumper.so">

File: localbot_description/urdf/localbot.urdf.xacro (robot description, xacro)
@@ -17,7 +17,13 @@
   <xacro:include filename="$(find localbot_description)/urdf/localbot.gazebo.macro.xacro"/>
   <xacro:gazebo_macro color="$(arg color)" laser_visual="false" camera_visual="false" imu_visual="true"/>
-  <link name="camera_support_link">
+  <link name="base_footprint"/>
+  <joint name="base_joint" type="fixed">
+    <parent link="base_footprint"/>
+    <child link="base_link" />
+    <origin xyz="0 0 0" rpy="0 0 0"/>
+  </joint>
+  <link name="base_link">
   </link>
-  <xacro:sensor_astra prefix="camera" parent="camera_support_link">
+  <xacro:sensor_astra prefix="camera" parent="base_link">
     <origin xyz="0.00 0.00 1.00" rpy="0 0.0 0" />
   </xacro:sensor_astra>
