Commit message: #6; add interactive marker to control the camera

File: localbot_description/urdf/localbot.urdf.xacro (robot description, xacro)
@@ -21,10 +21,10 @@
     <parent link="base_footprint"/>
     <child link="base_link" />
-    <origin xyz="0 0 0" rpy="0 0 0"/>
+    <origin xyz="0.00 0.00 0.00" rpy="0 0 0"/>
   </joint>
   <link name="base_link">
   </link>
   <xacro:sensor_astra prefix="camera" parent="base_link">
-    <origin xyz="0.00 0.00 1.00" rpy="0 0.0 0" />
+    <origin xyz="0.00 0.00 0.00" rpy="0 0.0 0" />
   </xacro:sensor_astra>
 </robot>

Commit message: #1; fix darkness in room_024.world

File: localbot_description/urdf/localbot.urdf.xacro (robot description, xacro)
@@ -12,7 +12,9 @@
   <xacro:property name="color" value="$(arg color)"/>
   <!-- Include other files-->
-  <xacro:include filename="$(find localbot_description)/urdf/properties.xacro"/>
-  <xacro:include filename="$(find localbot_description)/urdf/VLP-16.urdf.xacro"/>
+  <xacro:include filename="$(find hector_xacro_tools)/urdf/inertia_tensors.urdf.xacro" />
+  <xacro:include filename="$(find hector_xacro_tools)/urdf/joint_macros.urdf.xacro" />
+  <xacro:include filename="$(find hector_sensors_description)/urdf/kinect_camera.urdf.xacro" />
   <xacro:include filename="$(find localbot_description)/urdf/astra.urdf.xacro" />
+  <xacro:property name="M_PI" value="3.14159265359"/>
   <xacro:include filename="$(find localbot_description)/urdf/localbot.gazebo.macro.xacro"/>
   <xacro:gazebo_macro color="$(arg color)" laser_visual="false" camera_visual="false" imu_visual="true"/>
@@ -25,6 +27,9 @@
   <link name="base_link">
   </link>
-  <xacro:sensor_astra prefix="camera" parent="base_link">
+  <xacro:kinect_camera name='kinect' parent="base_link">
     <origin xyz="0.00 0.00 0.00" rpy="0 0.0 0" />
-  </xacro:sensor_astra>
+  </xacro:kinect_camera>
+  <!-- <xacro:sensor_astra prefix="back_camera" parent="base_link">
+    <origin xyz="0.0 0.00 0.00" rpy="0 0.0 0" />
+  </xacro:sensor_astra> -->
 </robot>
