Commit message: reorganize folders structure

File: synfeal_bringup/camera_description/urdf/astra.urdf.xacro (robot description, xacro)
@@ -17,5 +17,5 @@
         <origin xyz="-0.03 -0.06 0" rpy="${pi} 0 ${pi/2}"/>
         <geometry>
-          <mesh filename="package://localbot_description/meshes/astra2/astra2.dae" scale="1 1 1"/>
+          <mesh filename="package://synfeal_bringup/camera_description/meshes/astra2/astra2.dae" scale="1 1 1"/>
         </geometry>
       </visual>

File: synfeal_bringup/camera_description/urdf/localbot.urdf.xacro (robot description, xacro)
@@ -14,8 +14,8 @@
   <xacro:include filename="$(find hector_xacro_tools)/urdf/inertia_tensors.urdf.xacro" />
   <xacro:include filename="$(find hector_xacro_tools)/urdf/joint_macros.urdf.xacro" />
-  <xacro:include filename="$(find localbot_description)/urdf/localbot_kinect_camera.urdf.xacro" />
-  <!-- <xacro:include filename="$(find localbot_description)/urdf/atom_astra.urdf.xacro" /> -->
+  <xacro:include filename="$(find synfeal_bringup)/camera_description/urdf/localbot_kinect_camera.urdf.xacro" />
+  <!-- <xacro:include filename="$(find synfeal_bringup)/camera_description/urdf/atom_astra.urdf.xacro" /> -->
   <xacro:property name="M_PI" value="3.14159265359"/>
-  <xacro:include filename="$(find localbot_description)/urdf/localbot.gazebo.macro.xacro"/>
+  <xacro:include filename="$(find synfeal_bringup)/camera_description/urdf/localbot.gazebo.macro.xacro"/>
   <xacro:gazebo_macro color="$(arg color)" laser_visual="false" camera_visual="false" imu_visual="true"/>
   <link name="base_footprint"/>
