Commit message: added checks to verify if object is colliding with other objects

File: synfeal_bringup/camera_description/urdf/localbot_kinect_camera.urdf.xacro (robot description, xacro)
@@ -3,4 +3,7 @@
     <xacro:include filename="$(find hector_xacro_tools)/urdf/inertia_tensors.urdf.xacro"/>
     <xacro:property name="M_PI" value="3.1415926535897931" />
+    <material name="orange">
+      <color rgba="0.8 0.4 0.0 1.0"/>
+    </material>
     <xacro:macro name="kinect_camera_model" params="name parent *origin">
       <joint name="${name}_joint" type="fixed">
@@ -16,4 +19,5 @@
             <mesh filename="package://hector_sensors_description/meshes/kinect_camera/kinect_camera_simple.dae"/>
           </geometry>
+          <material name="orange"/>
         </visual>
         <collision>
