Commit message: added more objects

File: synfeal_bringup/camera_description/urdf/localbot.urdf.xacro (robot description, xacro)
@@ -19,4 +19,7 @@
   <xacro:include filename="$(find synfeal_bringup)/camera_description/urdf/localbot.gazebo.macro.xacro"/>
   <xacro:gazebo_macro color="$(arg color)" laser_visual="false" camera_visual="false" imu_visual="true"/>
+  <material name="marker_orange">
+    <color rgba= "0 0 1 1"/>
+  </material>
   <link name="base_footprint"/>
   <joint name="base_joint" type="fixed">
@@ -27,4 +30,24 @@
   <link name="base_link">
   </link>
+  <joint name="base_join" type="fixed">
+    <parent link="base_link"/>
+    <child link="marker_link" />
+    <origin xyz="0.00 0.00 0.20" rpy="0 0 0"/>
+  </joint>
+  <link name="marker_link">
+    <visual name="visual">
+      <geometry>
+        <box size="0.1 0.1 0.1" />
+      </geometry>
+      <material name="marker_orange"/>
+    </visual>
+    <visual name="visual">
+      <origin xyz="0.00 0.00 0.4" rpy="0 0 0"/>
+      <geometry>
+        <box size="0.1 0.1 0.4" />
+      </geometry>
+      <material name="marker_orange"/>
+    </visual>
+  </link>
   <xacro:kinect_camera name='kinect' parent="base_link">
     <origin xyz="0.00 0.00 0.00" rpy="0 0.0 0" />

Commit message: added option to reproduce camera movement from another dataset to data_collector

File: synfeal_bringup/camera_description/urdf/localbot.urdf.xacro (robot description, xacro)
@@ -20,5 +20,5 @@
   <xacro:gazebo_macro color="$(arg color)" laser_visual="false" camera_visual="false" imu_visual="true"/>
   <material name="marker_orange">
-    <color rgba= "0 0 1 1"/>
+    <color rgba="0.76 0.92 0.81 1"/>
   </material>
   <link name="base_footprint"/>
@@ -30,20 +30,13 @@
   <link name="base_link">
   </link>
-  <joint name="base_join" type="fixed">
+  <joint name="marker_joint" type="fixed">
     <parent link="base_link"/>
     <child link="marker_link" />
-    <origin xyz="0.00 0.00 0.20" rpy="0 0 0"/>
+    <origin xyz="0.00 0.00 0.25" rpy="1.57 0 1.57"/>
   </joint>
   <link name="marker_link">
-    <visual name="visual">
+    <visual>
       <geometry>
-        <box size="0.1 0.1 0.1" />
-      </geometry>
-      <material name="marker_orange"/>
-    </visual>
-    <visual name="visual">
-      <origin xyz="0.00 0.00 0.4" rpy="0 0 0"/>
-      <geometry>
-        <box size="0.1 0.1 0.4" />
+        <mesh filename="package://synfeal_bringup/camera_description/meshes/cameraicon/frustum.obj"/>
       </geometry>
       <material name="marker_orange"/>

Commit message: added frustum to the camera

File: synfeal_bringup/camera_description/urdf/localbot.urdf.xacro (robot description, xacro)
@@ -33,14 +33,33 @@
     <parent link="base_link"/>
     <child link="marker_link" />
-    <origin xyz="0.00 0.00 0.25" rpy="1.57 0 1.57"/>
+    <origin xyz="0.01 0.00 0.00" rpy="1.57 0 -1.57"/>
   </joint>
   <link name="marker_link">
     <visual>
+      <transparency>1</transparency>
       <geometry>
-        <mesh filename="package://synfeal_bringup/camera_description/meshes/cameraicon/frustum.obj"/>
+        <mesh filename="package://synfeal_bringup/camera_description/meshes/cameraicon/frustrum_frame.obj"/>
       </geometry>
-      <material name="marker_orange"/>
     </visual>
   </link>
+  <joint name="marker_inside_joint" type="fixed">
+    <parent link="marker_link"/>
+    <child link="marker_inside_link" />
+    <origin xyz="0.00 0.00 0.00" rpy="0 0 0"/>
+  </joint>
+  <link name="marker_inside_link">
+    <visual>
+      <transparency>1</transparency>
+      <geometry>
+        <mesh filename="package://synfeal_bringup/camera_description/meshes/cameraicon/frustrum.obj"/>
+      </geometry>
+    </visual>
+  </link>
+  <gazebo reference="marker_link">
+    <material>Gazebo/BlackTransparent</material>
+  </gazebo>
+  <gazebo reference="marker_inside_link">
+    <material>Gazebo/GreyTransparent</material>
+  </gazebo>
   <xacro:kinect_camera name='kinect' parent="base_link">
     <origin xyz="0.00 0.00 0.00" rpy="0 0.0 0" />
